Commit message: Robotun önüne hizalandı

File: urdf/custom_husky.urdf.xacro (robot description, xacro)
@@ -28,5 +28,5 @@
   <joint name="camera_joint" type="fixed">
     <axis xyz="0 1 0"/>
-    <origin xyz="0.3 0 0.3" rpy="0 0 0"/>
+    <origin xyz="0.3 0 0.0" rpy="0 0 0"/>
     <parent link="top_plate_link"/>
     <child link="camera_link"/>

Commit message: IRO içindeyse locationla çakışcaz

File: urdf/custom_husky.urdf.xacro (robot description, xacro)
@@ -1,76 +1,76 @@
 <?xml version="1.0"?>
 <robot name="husky" xmlns:xacro="http://ros.org/wiki/xacro">
-  <!-- Include the base Husky URDF -->
-  <xacro:include filename="$(find husky_description)/urdf/husky.urdf.xacro" />
-  <!-- Camera Link -->
-  <link name="camera_link">
-    <visual>
-      <origin xyz="0 0 0" rpy="0 0 0"/>
-      <geometry>
-        <box size="0.1 0.1 0.1"/>
-      </geometry>
-      <material name="red">
-        <color rgba="1 0 0 1"/>
-      </material>
-    </visual>
-    <collision>
-      <origin xyz="0 0 0" rpy="0 0 0"/>
-      <geometry>
-        <box size="0.1 0.1 0.1"/>
-      </geometry>
-    </collision>
-    <inertial>
-      <mass value="1e-5"/>
-      <origin xyz="0 0 0" rpy="0 0 0"/>
-      <inertia ixx="1e-6" ixy="0" ixz="0" iyy="1e-6" iyz="0" izz="1e-6"/>
-    </inertial>
-  </link>
-  <joint name="camera_joint" type="fixed">
-    <axis xyz="0 1 0"/>
-    <origin xyz="0.3 0 0.0" rpy="0 0 0"/>
-    <parent link="top_plate_link"/>
-    <child link="camera_link"/>
-  </joint>
-  <gazebo reference="camera_link">
-    <material>Gazebo/Red</material>
-    <turnGravityOff>false</turnGravityOff>
-    <selfCollide>false</selfCollide>
-  </gazebo>
-  <gazebo reference="camera_link">
-    <sensor type="depth" name="camera">
-      <always_on>true</always_on>
-      <update_rate>30.0</update_rate>
-      <camera>
-        <horizontal_fov>1.047198</horizontal_fov>
-        <image>
-          <width>640</width>
-          <height>480</height>
-          <format>R8G8B8</format>
-        </image>
-        <clip>
-          <near>0.05</near>
-          <far>10.0</far>
-        </clip>
-      </camera>
-      <plugin name="kinect_camera_controller" filename="libgazebo_ros_openni_kinect.so">
-        <baseline>0.2</baseline>
-        <alwaysOn>true</alwaysOn>
-        <updateRate>30.0</updateRate>
-        <cameraName>camera</cameraName>
-        <imageTopicName>rgb/image_raw</imageTopicName>
-        <cameraInfoTopicName>rgb/camera_info</cameraInfoTopicName>
-        <depthImageTopicName>depth/image_raw</depthImageTopicName>
-        <depthImageInfoTopicName>depth/camera_info</depthImageInfoTopicName>
-        <pointCloudTopicName>depth/points</pointCloudTopicName>
-        <frameName>camera_link</frameName>
-        <pointCloudCutoff>0.5</pointCloudCutoff>
-        <pointCloudCutoffMax>10.0</pointCloudCutoffMax>
-        <distortionK1>0.00000001</distortionK1>
-        <distortionK2>0.00000001</distortionK2>
-        <distortionK3>0.00000001</distortionK3>
-        <distortionT1>0.00000001</distortionT1>
-        <distortionT2>0.00000001</distortionT2>
-      </plugin>
-    </sensor>
-  </gazebo>
+    <!-- Husky robot tanımı -->
+    <xacro:arg name="laser_enabled" default="false"/>
+    <xacro:arg name="laser_xyz" default="$(optenv HUSKY_LMS1XX_XYZ 0.2206 0.0 0.00635)"/>
+    <xacro:arg name="laser_rpy" default="$(optenv HUSKY_LMS1XX_RPY 0.0 0.0 0.0)"/>
+    <!-- Include Husky URDF -->
+    <xacro:include filename="$(find husky_description)/urdf/husky.urdf.xacro" />
+    <!-- Camera Link -->
+    <link name="camera_link">
+        <collision>
+            <origin xyz="0 0 0" rpy="0 0 0"/>
+            <geometry>
+                <box size="0.1 0.1 0.1"/>
+            </geometry>
+        </collision>
+        <visual>
+            <origin xyz="0 0 0" rpy="0 0 0"/>
+            <geometry>
+                <box size="0.1 0.1 0.1"/>
+            </geometry>
+            <material name="red">
+                <color rgba="1 0 0 1"/>
+            </material>
+        </visual>
+        <inertial>
+            <mass value="1e-5"/>
+            <origin xyz="0 0 0" rpy="0 0 0"/>
+            <inertia ixx="1e-6" ixy="0" ixz="0" iyy="1e-6" iyz="0" izz="1e-6"/>
+        </inertial>
+    </link>
+    <!-- Camera Joint -->
+    <joint name="camera_joint" type="fixed">
+        <axis xyz="0 1 0"/>
+        <origin xyz="0.3 0 0.1" rpy="0 0 0"/>
+        <parent link="top_plate_link"/>
+        <child link="camera_link"/>
+    </joint>
+    <!-- Gazebo Tags -->
+    <gazebo reference="camera_link">
+        <material>Gazebo/Red</material>
+    </gazebo>
+    <!-- Depth Camera Plugin -->
+    <gazebo reference="camera_link">
+        <sensor type="depth" name="camera">
+            <always_on>true</always_on>
+            <update_rate>30.0</update_rate>
+            <camera>
+                <horizontal_fov>1.5708</horizontal_fov>
+                <image>
+                    <width>848</width>
+                    <height>480</height>
+                    <format>R8G8B8</format>
+                </image>
+                <clip>
+                    <near>0.05</near>
+                    <far>15.0</far>
+                </clip>
+            </camera>
+            <plugin name="kinect_camera_controller" filename="libgazebo_ros_openni_kinect.so">
+                <alwaysOn>true</alwaysOn>
+                <updateRate>30.0</updateRate>
+                <cameraName>camera</cameraName>
+                <frameName>camera_link</frameName>
+                <imageTopicName>rgb/image_raw</imageTopicName>
+                <cameraInfoTopicName>rgb/camera_info</cameraInfoTopicName>
+                <depthImageTopicName>depth/image_raw</depthImageTopicName>
+                <depthImageInfoTopicName>depth/camera_info</depthImageInfoTopicName>
+                <pointCloudTopicName>depth/points</pointCloudTopicName>
+                <pointCloudCutoff>0.3</pointCloudCutoff>
+                <pointCloudCutoffMax>15.0</pointCloudCutoffMax>
+                <rangeMax>15.0</rangeMax>
+            </plugin>
+        </sensor>
+    </gazebo>
 </robot>
